Commit message: adding gazebo support

File: config/so101_new_calib.ros2_control.xacro (robot description, xacro)
@@ -5,6 +5,5 @@
         <ros2_control name="${name}" type="system">
             <hardware>
-                <!-- By default, set up controllers for simulation. This won't work on real hardware -->
-                <plugin>mock_components/GenericSystem</plugin>
+                <plugin>gz_ros2_control/GazeboSimSystem</plugin>
             </hardware>
             <joint name="shoulder_pan">

File: config/so101_new_calib.urdf.xacro (robot description, xacro)
@@ -6,4 +6,24 @@
     <!-- Import control_xacro -->
     <xacro:include filename="so101_new_calib.ros2_control.xacro" />
-    <xacro:so101_new_calib_ros2_control name="FakeSystem" initial_positions_file="$(arg initial_positions_file)"/>
+    <!-- World link anchor for Gazebo physics -->
+    <link name="world"/>
+    <joint name="world_base_joint" type="fixed">
+        <parent link="world"/>
+        <child link="base_link"/>
+        <origin xyz="0 0 0" rpy="0 0 0"/>
+    </joint>
+    <gazebo reference="world_base_joint">
+        <preserveFixedJoint>true</preserveFixedJoint>
+    </gazebo>
+    <!-- Gazebo-side mount constraint: keep the base fixed against gravity/torque loads. -->
+    <gazebo reference="base_link">
+        <gravity>false</gravity>
+        <kinematic>true</kinematic>
+    </gazebo>
+    <xacro:so101_new_calib_ros2_control name="GazeboSimSystem" initial_positions_file="$(arg initial_positions_file)"/>
+    <gazebo>
+        <plugin filename="libgz_ros2_control-system.so" name="gz_ros2_control::GazeboSimROS2ControlPlugin">
+            <parameters>$(find so101_moveit_config)/config/ros2_controllers.yaml</parameters>
+        </plugin>
+    </gazebo>
 </robot>

Commit message: adding camera

File: config/so101_new_calib.ros2_control.xacro (robot description, xacro)
@@ -2,5 +2,5 @@
 <robot xmlns:xacro="http://www.ros.org/wiki/xacro">
     <xacro:macro name="so101_new_calib_ros2_control" params="name initial_positions_file">
-        <xacro:property name="initial_positions" value="${load_yaml(initial_positions_file)['initial_positions']}"/>
+    <xacro:property name="initial_positions" value="${xacro.load_yaml(initial_positions_file)['initial_positions']}"/>
         <ros2_control name="${name}" type="system">
             <hardware>
